File: Main.sch (EAGLE design)
At the start: 27 parts, among them U1 L298, U2 LM 1085 IT5,0, U3 LM 1085 IT3,3, U4 L298, X1 12V

Commit message: using ria screw terminals
Parts:
- removed X2: (no value), con-wago255:233-504
- added X3: Battery, con-ria-59:AKL59-02
- SV1: value (none) -> Raspberry Pi B Plus Connector
- U2: value LM 1085 IT5,0 -> LM 1084 IT5,0; device linear-technology-3:LT1085IT-V -> v-reg-2:LM1084-V
- U3: value LM 1085 IT3,3 -> LM 1084 IT3,3; device linear-technology-3:LT1085IT-V -> v-reg-2:LM1084-V
- X1: value 12V -> Motors; device con-wago-508:W237-02P -> con-ria-59:AKL59-08
Connections:
- net GND: now also X3-2.1; no longer X1-2.KL
- net ML_OUT_A: now also X1-1.1, X1-3.1; no longer X2.-1
- net ML_OUT_B: now also X1-2.1, X1-4.1; no longer X2.-2
- net MR_OUT_A: now also X1-5.1, X1-7.1; no longer X2.-3
- net MR_OUT_B: now also X1-6.1, X1-8.1; no longer X2.-4
- net N$1: now also X3-1.1; no longer X1-1.KL
Other:
- moved on the sheet: SV1, X1-1, X1-2
Changed lines of the file:
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@@
 </classes>
 <parts>
-<part name="U2" library="linear-technology-3" deviceset="LT1085*" device="T-V" technology="I" value="LM 1085 IT5,0"/>
+<part name="U2" library="v-reg-2" deviceset="LM1084" device="-V" value="LM 1084 IT5,0"/>
 <part name="D5" library="semicon-smd-ipc" deviceset="D-" device="MLL-41" value="1N4007"/>
 <part name="C1" library="rcl" deviceset="C-EU" device="025-040X050" value="10uF Tant."/>
 <part name="C2" library="rcl" deviceset="C-EU" device="025-040X050" value="10uF Tant."/>
-<part name="X1" library="con-wago-508" deviceset="W237-02P" device="" value="12V"/>
-<part name="U3" library="linear-technology-3" deviceset="LT1085*" device="T-V" technology="I" value="LM 1085 IT3,3"/>
+<part name="U3" library="v-reg-2" deviceset="LM1084" device="-V" value="LM 1084 IT3,3"/>
 <part name="D6" library="semicon-smd-ipc" deviceset="D-" device="MLL-41" value="1N4007"/>
 <part name="C4" library="rcl" deviceset="C-EU" device="025-040X050" value="10uF Tant."/>
@@
 <part name="GND1" library="supply1" deviceset="GND" device=""/>
 <part name="GND3" library="supply1" deviceset="GND" device=""/>
-<part name="X2" library="con-wago255" deviceset="233-504" device=""/>
-<part name="SV1" library="con-lsta" deviceset="FE20-2" device=""/>
+<part name="SV1" library="con-lsta" deviceset="FE20-2" device="" value="Raspberry Pi B Plus Connector"/>
 <part name="GND4" library="supply1" deviceset="GND" device=""/>
 <part name="D2" library="diode" deviceset="P600" device="" value="1N4007"/>
@@
 <part name="GND7" library="supply1" deviceset="GND" device=""/>
 <part name="GND8" library="supply1" deviceset="GND" device=""/>
+<part name="FRAME3" library="frames" deviceset="DINA4_L" device=""/>
+<part name="FRAME4" library="frames" deviceset="DINA4_L" device=""/>
+<part name="X3" library="con-ria-59" deviceset="AKL59-02" device="" value="Battery"/>
+<part name="X1" library="con-ria-59" deviceset="AKL59-08" device="" value="Motors"/>
 </parts>
 <sheets>
@@
 <instance part="C1" gate="G$1" x="-429.26" y="297.18"/>
 <instance part="C2" gate="G$1" x="-393.7" y="332.74"/>
-<instance part="X1" gate="-1" x="-492.76" y="340.36"/>
-<instance part="X1" gate="-2" x="-492.76" y="325.12"/>
 <instance part="U3" gate="G$1" x="-411.48" y="304.8"/>
 <instance part="D6" gate="G$1" x="-411.48" y="317.5" rot="MR0"/>
@@
 <instance part="GND1" gate="1" x="-459.74" y="312.42"/>
 <instance part="GND3" gate="1" x="-487.68" y="137.16"/>
-<instance part="X2" gate="G$1" x="-261.62" y="124.46"/>
-<instance part="SV1" gate="G$1" x="-299.72" y="322.58"/>
-<instance part="GND4" gate="1" x="-281.94" y="299.72"/>
+<instance part="SV1" gate="G$1" x="-388.62" y="518.16"/>
+<instance part="GND4" gate="1" x="-370.84" y="495.3"/>
 <instance part="D2" gate="G$1" x="-381" y="167.64" rot="R90"/>
 <instance part="D3" gate="G$1" x="-398.78" y="167.64" rot="R90"/>
@@
 <instance part="GND7" gate="1" x="-398.78" y="71.12"/>
 <instance part="GND8" gate="1" x="-381" y="71.12"/>
+<instance part="FRAME3" gate="G$1" x="-513.08" y="408.94"/>
+<instance part="FRAME3" gate="G$2" x="-350.52" y="408.94"/>
+<instance part="FRAME4" gate="G$1" x="-513.08" y="-172.72"/>
+<instance part="FRAME4" gate="G$2" x="-350.52" y="-172.72"/>
+<instance part="X3" gate="-1" x="-487.68" y="340.36" rot="MR0"/>
+<instance part="X3" gate="-2" x="-487.68" y="325.12" rot="MR0"/>
+<instance part="X1" gate="-1" x="-327.66" y="139.7"/>
+<instance part="X1" gate="-2" x="-327.66" y="134.62"/>
+<instance part="X1" gate="-3" x="-327.66" y="129.54"/>
+<instance part="X1" gate="-4" x="-327.66" y="124.46"/>
+<instance part="X1" gate="-5" x="-327.66" y="119.38"/>
+<instance part="X1" gate="-6" x="-327.66" y="114.3"/>
+<instance part="X1" gate="-7" x="-327.66" y="109.22"/>
+<instance part="X1" gate="-8" x="-327.66" y="104.14"/>
 </instances>
 <busses>
@@
 <net name="N$1" class="0">
 <segment>
-<pinref part="X1" gate="-1" pin="KL"/>
 <pinref part="F1" gate="G$1" pin="1"/>
 <wire x1="-487.68" y1="340.36" x2="-480.06" y2="340.36" width="0.1524" layer="91"/>
+<pinref part="X3" gate="-1" pin="1"/>
 </segment>
 </net>
@@
 <wire x1="-447.04" y1="289.56" x2="-447.04" y2="325.12" width="0.1524" layer="91"/>
 <junction x="-447.04" y="325.12"/>
-<pinref part="X1" gate="-2" pin="KL"/>
 <wire x1="-487.68" y1="325.12" x2="-459.74" y2="325.12" width="0.1524" layer="91"/>
 <pinref part="C2" gate="G$1" pin="2"/>
@@
 <junction x="-429.26" y="325.12"/>
 <pinref part="GND1" gate="1" pin="GND"/>
+<pinref part="X3" gate="-2" pin="1"/>
 </segment>
 <segment>
 <pinref part="SV1" gate="G$1" pin="6"/>
 <pinref part="GND4" gate="1" pin="GND"/>
-<wire x1="-292.1" y1="302.26" x2="-281.94" y2="302.26" width="0.1524" layer="91"/>
+<wire x1="-381" y1="497.84" x2="-370.84" y2="497.84" width="0.1524" layer="91"/>
 </segment>
 <segment>
@@
 </segment>
 <segment>
-<pinref part="X2" gate="G$1" pin="-2"/>
-<wire x1="-269.24" y1="124.46" x2="-274.32" y2="124.46" width="0.1524" layer="91"/>
+<pinref part="X1" gate="-2" pin="1"/>
+<wire x1="-327.66" y1="134.62" x2="-332.74" y2="134.62" width="0.1524" layer="91"/>
+<label x="-340.36" y="134.62" size="1.778" layer="95"/>
+</segment>
+<segment>
+<pinref part="X1" gate="-4" pin="1"/>
+<wire x1="-327.66" y1="124.46" x2="-332.74" y2="124.46" width="0.1524" layer="91"/>
+<label x="-340.36" y="124.46" size="1.778" layer="95"/>
 </segment>
 </net>
@@
 </segment>
 <segment>
-<pinref part="X2" gate="G$1" pin="-1"/>
-<wire x1="-269.24" y1="127" x2="-274.32" y2="127" width="0.1524" layer="91"/>
+<pinref part="X1" gate="-1" pin="1"/>
+<wire x1="-327.66" y1="139.7" x2="-332.74" y2="139.7" width="0.1524" layer="91"/>
+<label x="-340.36" y="139.7" size="1.778" layer="95"/>
+</segment>
+<segment>
+<pinref part="X1" gate="-3" pin="1"/>
+<wire x1="-327.66" y1="129.54" x2="-332.74" y2="129.54" width="0.1524" layer="91"/>
+<label x="-340.36" y="129.54" size="1.778" layer="95"/>
 </segment>
 </net>
@@
 </segment>
 <segment>
-<pinref part="X2" gate="G$1" pin="-3"/>
-<wire x1="-269.24" y1="121.92" x2="-274.32" y2="121.92" width="0.1524" layer="91"/>
+<pinref part="X1" gate="-5" pin="1"/>
+<wire x1="-327.66" y1="119.38" x2="-332.74" y2="119.38" width="0.1524" layer="91"/>
+<label x="-340.36" y="119.38" size="1.778" layer="95"/>
+</segment>
+<segment>
+<pinref part="X1" gate="-7" pin="1"/>
+<wire x1="-327.66" y1="109.22" x2="-332.74" y2="109.22" width="0.1524" layer="91"/>
+<label x="-340.36" y="109.22" size="1.778" layer="95"/>
 </segment>
 </net>
@@
 </segment>
 <segment>
-<pinref part="X2" gate="G$1" pin="-4"/>
-<wire x1="-269.24" y1="119.38" x2="-274.32" y2="119.38" width="0.1524" layer="91"/>
-</segment>
-</net>
+<pinref part="X1" gate="-6" pin="1"/>
+<wire x1="-327.66" y1="114.3" x2="-332.74" y2="114.3" width="0.1524" layer="91"/>
+<label x="-340.36" y="114.3" size="1.778" layer="95"/>
+</segment>
+<segment>
+<pinref part="X1" gate="-8" pin="1"/>
+<wire x1="-327.66" y1="104.14" x2="-332.74" y2="104.14" width="0.1524" layer="91"/>
+<label x="-340.36" y="104.14" size="1.778" layer="95"/>
+</segment>
+</net>
