File: Main.sch (EAGLE design)
At the start: 39 parts, among them Q1 IRF9530, U1 L298, U2 LM 1084 IT5,0, U3 LM 1084 IT3,3, U4 L298, X1 Motors, X2 PIRs, X3 Battery

Commit message: ?
Parts:
- X4: value (none) -> Ultra Sonics
Other:
- moved on the sheet: R3, R5, X4
Changed lines of the file:
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@@
 <part name="F5" library="_hhn_PtcFuses_Siba_r500" deviceset="SIBA194600*" device="" value="PTC194600-150"/>
 <part name="F6" library="_hhn_PtcFuses_Siba_r500" deviceset="SIBA194600*" device="" value="PTC194600-150"/>
-<part name="X4" library="con-wago" deviceset="233-508" device=""/>
+<part name="X4" library="con-wago" deviceset="233-508" device="" value="Ultra Sonics"/>
 <part name="R2" library="resistor" deviceset="R-EU_" device="R0805" value="330"/>
 <part name="R3" library="resistor" deviceset="R-EU_" device="R0805" value="470"/>
@@
 <instance part="F5" gate="G$1" x="-292.1" y="121.92"/>
 <instance part="F6" gate="G$1" x="-292.1" y="111.76"/>
-<instance part="X4" gate="G$1" x="-360.68" y="-30.48"/>
+<instance part="X4" gate="G$1" x="-355.6" y="-30.48"/>
 <instance part="R2" gate="G$1" x="-381" y="-27.94" rot="R180"/>
-<instance part="R3" gate="G$1" x="-398.78" y="-27.94" rot="R180"/>
+<instance part="R3" gate="G$1" x="-403.86" y="-27.94" rot="R180"/>
 <instance part="R4" gate="G$1" x="-381" y="-38.1" rot="R180"/>
-<instance part="R5" gate="G$1" x="-398.78" y="-38.1" rot="R180"/>
+<instance part="R5" gate="G$1" x="-403.86" y="-38.1" rot="R180"/>
 <instance part="GND10" gate="1" x="-414.02" y="-60.96"/>
 </instances>
@@
 <segment>
 <pinref part="X4" gate="G$1" pin="B-1"/>
-<wire x1="-368.3" y1="-22.86" x2="-426.72" y2="-22.86" width="0.1524" layer="91"/>
+<wire x1="-363.22" y1="-22.86" x2="-426.72" y2="-22.86" width="0.1524" layer="91"/>
 <wire x1="-426.72" y1="-22.86" x2="-426.72" y2="-33.02" width="0.1524" layer="91"/>
 <pinref part="X4" gate="G$1" pin="B-5"/>
 <wire x1="-426.72" y1="-33.02" x2="-426.72" y2="-60.96" width="0.1524" layer="91"/>
-<wire x1="-368.3" y1="-33.02" x2="-426.72" y2="-33.02" width="0.1524" layer="91"/>
+<wire x1="-363.22" y1="-33.02" x2="-426.72" y2="-33.02" width="0.1524" layer="91"/>
 <junction x="-426.72" y="-33.02"/>
 <label x="-426.72" y="-63.5" size="1.778" layer="95"/>
@@
 <segment>
 <pinref part="R3" gate="G$1" pin="2"/>
-<wire x1="-403.86" y1="-27.94" x2="-414.02" y2="-27.94" width="0.1524" layer="91"/>
+<wire x1="-408.94" y1="-27.94" x2="-414.02" y2="-27.94" width="0.1524" layer="91"/>
 <wire x1="-414.02" y1="-27.94" x2="-414.02" y2="-30.48" width="0.1524" layer="91"/>
 <pinref part="R5" gate="G$1" pin="2"/>
@@
 <wire x1="-414.02" y1="-38.1" x2="-414.02" y2="-40.64" width="0.1524" layer="91"/>
 <wire x1="-414.02" y1="-40.64" x2="-414.02" y2="-58.42" width="0.1524" layer="91"/>
-<wire x1="-403.86" y1="-38.1" x2="-414.02" y2="-38.1" width="0.1524" layer="91"/>
+<wire x1="-408.94" y1="-38.1" x2="-414.02" y2="-38.1" width="0.1524" layer="91"/>
 <junction x="-414.02" y="-38.1"/>
 <pinref part="GND10" gate="1" pin="GND"/>
 <pinref part="X4" gate="G$1" pin="B-8"/>
-<wire x1="-368.3" y1="-40.64" x2="-414.02" y2="-40.64" width="0.1524" layer="91"/>
+<wire x1="-363.22" y1="-40.64" x2="-414.02" y2="-40.64" width="0.1524" layer="91"/>
 <junction x="-414.02" y="-40.64"/>
 <pinref part="X4" gate="G$1" pin="B-4"/>
-<wire x1="-368.3" y1="-30.48" x2="-414.02" y2="-30.48" width="0.1524" layer="91"/>
+<wire x1="-363.22" y1="-30.48" x2="-414.02" y2="-30.48" width="0.1524" layer="91"/>
 <junction x="-414.02" y="-30.48"/>
 </segment>
@@
 <pinref part="X4" gate="G$1" pin="B-3"/>
 <pinref part="R2" gate="G$1" pin="1"/>
-<wire x1="-368.3" y1="-27.94" x2="-375.92" y2="-27.94" width="0.1524" layer="91"/>
+<wire x1="-363.22" y1="-27.94" x2="-375.92" y2="-27.94" width="0.1524" layer="91"/>
 </segment>
 </net>
@@
 <pinref part="R3" gate="G$1" pin="1"/>
 <wire x1="-386.08" y1="-27.94" x2="-393.7" y2="-27.94" width="0.1524" layer="91"/>
+<wire x1="-393.7" y1="-27.94" x2="-398.78" y2="-27.94" width="0.1524" layer="91"/>
 <wire x1="-393.7" y1="-27.94" x2="-393.7" y2="-60.96" width="0.1524" layer="91"/>
 <junction x="-393.7" y="-27.94"/>
@@
 <pinref part="R5" gate="G$1" pin="1"/>
 <wire x1="-386.08" y1="-38.1" x2="-388.62" y2="-38.1" width="0.1524" layer="91"/>
-<wire x1="-388.62" y1="-38.1" x2="-393.7" y2="-38.1" width="0.1524" layer="91"/>
+<wire x1="-388.62" y1="-38.1" x2="-398.78" y2="-38.1" width="0.1524" layer="91"/>
 <wire x1="-388.62" y1="-38.1" x2="-388.62" y2="-60.96" width="0.1524" layer="91"/>
 <junction x="-388.62" y="-38.1"/>
@@
 <pinref part="R4" gate="G$1" pin="1"/>
 <pinref part="X4" gate="G$1" pin="B-7"/>
-<wire x1="-375.92" y1="-38.1" x2="-368.3" y2="-38.1" width="0.1524" layer="91"/>
+<wire x1="-375.92" y1="-38.1" x2="-363.22" y2="-38.1" width="0.1524" layer="91"/>
 </segment>
 </net>
@@
 <segment>
 <pinref part="X4" gate="G$1" pin="B-2"/>
-<wire x1="-368.3" y1="-25.4" x2="-373.38" y2="-25.4" width="0.1524" layer="91"/>
+<wire x1="-363.22" y1="-25.4" x2="-373.38" y2="-25.4" width="0.1524" layer="91"/>
 <wire x1="-373.38" y1="-25.4" x2="-373.38" y2="-60.96" width="0.1524" layer="91"/>
 <label x="-373.38" y="-60.96" size="1.778" layer="95" rot="R90"/>
@@
 <net name="USM_B_TRIG" class="0">
 <segment>
-<pinref part="X4" gate="G$1" pin="B-6"/>
-<wire x1="-368.3" y1="-35.56" x2="-368.3" y2="-60.96" width="0.1524" layer="91"/>
-<label x="-368.3" y="-60.96" size="1.778" layer="95" rot="R90"/>
-</segment>
-<segment>
 <pinref part="SV1" gate="G$1" pin="16"/>
 <wire x1="-381" y1="510.54" x2="-355.6" y2="510.54" width="0.1524" layer="91"/>
 <label x="-355.6" y="510.54" size="1.778" layer="95"/>
 </segment>
-</net>
+<segment>
+<pinref part="X4" gate="G$1" pin="B-6"/>
+<wire x1="-363.22" y1="-35.56" x2="-368.3" y2="-35.56" width="0.1524" layer="91"/>
+<wire x1="-368.3" y1="-35.56" x2="-368.3" y2="-60.96" width="0.1524" layer="91"/>
+<label x="-368.3" y="-60.96" size="1.778" layer="95" rot="R90"/>
+</segment>
+</net>

Commit message: a third ultrasonic sensor
Parts:
- added R6: 470, resistor:R-EU_R0805
- added R7: 330, resistor:R-EU_R0805
- R2, R4: value 330 -> 470
- R3, R5: value 470 -> 330
Connections:
- removed net N$16: R2.1, X4.B-3
- removed net N$25: SV1.13
- removed net N$28: SV1.19
- removed net N$35: R4.1, X4.B-7
- new net N$22: R7.1, X4.B-2
- new net N$24: R3.1, X4.B-4
- new net N$33: R5.1, X4.B-6
- new net USM_C_ECHO: R4.1, R5.2, SV1.13
- new net USM_C_TRIG: SV1.19, X4.B-5
- net +5V: now also X4.B-7; no longer X4.B-1, X4.B-5
- net GND: now also R2.2, R4.2, R6.2; no longer R3.2, R5.2, X4.B-4
- net USM_A_ECHO: now also R6.1, R7.2; no longer R2.2, R3.1
- net USM_A_TRIG: now also X4.B-1; no longer X4.B-2
- net USM_B_ECHO: now also R2.1, R3.2; no longer R4.2, R5.1
- net USM_B_TRIG: now also X4.B-3; no longer X4.B-6
Other:
- moved on the sheet: R2, R3, R4, R5, X4
